File: pcb/aquarium.sch (EAGLE design)
At the start: 54 parts, among them J1 PUMP_PWR, J10 DO_IN, J11 LD1117, J12 LEVEL, J13 FLOW, J14 5V_INPUT, J15 DO, J16 PH, J17 EC_IN, J18 EC, J19 EC_PWR_OUT, J2 EC_OUT, J20 EC_PWR_IN, J21 MCP3424-B, J22 MCP3424-A, J24 ADC-3, J25 ADC-4, J26 DS18B20, J27 DS18B20, J28 LD1117, J3 PH_PWR_OUT, J4 PH_PWR_IN, J5 DO_PWR_OUT, J6 DO_PWR_IN, J7 PH_OUT, J8 DO_OUT, J9 PH_IN, Q1 2n3904, Q2 2n3904, Q3 2n3904, Q4 2n3904

Commit message: Bumping some things
* Minor updates to main
* Fixing PCB and schematic
Parts:
- added J23: GPIO, SparkFun-Connectors:CONN_02
Connections:
- new net GPIO_11: J23.1, ONION.I2S_CLK/GPIO3
- net GND: now also J23.2
Changed lines of the file:
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@@
 <part name="GND24" library="supply1" library_urn="urn:adsk.eagle:library:371" deviceset="GND" device=""/>
 <part name="GND25" library="supply1" library_urn="urn:adsk.eagle:library:371" deviceset="GND" device=""/>
+<part name="J23" library="SparkFun-Connectors" library_urn="urn:adsk.eagle:library:513" deviceset="CONN_02" device="" package3d_urn="urn:adsk.eagle:package:38039/1" value="GPIO"/>
+<part name="GND26" library="supply1" library_urn="urn:adsk.eagle:library:371" deviceset="GND" device=""/>
 </parts>
 <sheets>
@@
 <instance part="GND25" gate="1" x="137.16" y="22.86" smashed="yes">
 <attribute name="VALUE" x="138.176" y="16.51" size="1.778" layer="96" rot="R90"/>
+</instance>
+<instance part="J23" gate="G$1" x="99.06" y="132.08" smashed="yes" rot="R270">
+<attribute name="VALUE" x="94.234" y="134.62" size="1.778" layer="96" font="vector" rot="R270"/>
+<attribute name="NAME" x="104.648" y="134.62" size="1.778" layer="95" font="vector" rot="R270"/>
+</instance>
+<instance part="GND26" gate="1" x="101.6" y="109.22" smashed="yes">
+<attribute name="VALUE" x="99.06" y="106.68" size="1.778" layer="96"/>
 </instance>
 </instances>
@@
 <wire x1="137.16" y1="38.1" x2="137.16" y2="25.4" width="0.1524" layer="91"/>
 <pinref part="GND25" gate="1" pin="GND"/>
+</segment>
+<segment>
+<pinref part="J23" gate="G$1" pin="2"/>
+<wire x1="101.6" y1="124.46" x2="101.6" y2="111.76" width="0.1524" layer="91"/>
+<pinref part="GND26" gate="1" pin="GND"/>
 </segment>
 </net>
@@
 </segment>
 </net>
+<net name="GPIO_11" class="0">
+<segment>
+<pinref part="ONION" gate="OMEGA2+" pin="I2S_CLK/GPIO3"/>
+<wire x1="314.96" y1="226.06" x2="294.64" y2="226.06" width="0.1524" layer="91"/>
+<label x="294.64" y="226.06" size="1.016" layer="95" rot="R180" xref="yes"/>
+</segment>
+<segment>
+<pinref part="J23" gate="G$1" pin="1"/>
+<wire x1="99.06" y1="124.46" x2="99.06" y2="119.38" width="0.1524" layer="91"/>
+<label x="99.06" y="119.38" size="1.016" layer="95" rot="R270" xref="yes"/>
+</segment>
+</net>

Commit message: Updating PCB design to latest
Connections:
- net GND: now also J12.3, J24.3, J25.3; no longer J12.2, J24.2, J25.2
- net VDD: now also J12.2, J24.2, J25.2; no longer J12.3, J24.3, J25.3
Changed lines of the file:
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@@
 <?xml version="1.0" encoding="utf-8"?>
 <!DOCTYPE eagle SYSTEM "eagle.dtd">
-<eagle version="9.5.1">
+<eagle version="9.5.2">
 <drawing>
 <settings>
@@
 <attribute name="VALUE" x="180.34" y="96.52" size="1.778" layer="96"/>
 </instance>
-<instance part="VDD7" gate="G$1" x="139.7" y="109.22" smashed="yes" rot="R180">
-<attribute name="VALUE" x="139.7" y="106.68" size="1.778" layer="96" rot="R270"/>
+<instance part="VDD7" gate="G$1" x="137.16" y="109.22" smashed="yes" rot="R180">
+<attribute name="VALUE" x="137.16" y="106.68" size="1.778" layer="96" rot="R270"/>
 </instance>
 <instance part="H1" gate="G$1" x="48.26" y="40.64" smashed="yes">
@@
 <attribute name="NAME" x="142.748" y="48.26" size="1.778" layer="95" font="vector" rot="R270"/>
 </instance>
-<instance part="VDD12" gate="G$1" x="121.92" y="25.4" smashed="yes" rot="R180">
-<attribute name="VALUE" x="124.46" y="27.94" size="1.778" layer="96" rot="R270"/>
-</instance>
-<instance part="VDD13" gate="G$1" x="139.7" y="25.4" smashed="yes" rot="R180">
-<attribute name="VALUE" x="142.24" y="27.94" size="1.778" layer="96" rot="R270"/>
+<instance part="VDD12" gate="G$1" x="119.38" y="25.4" smashed="yes" rot="R180">
+<attribute name="VALUE" x="118.618" y="21.844" size="1.778" layer="96" rot="R270"/>
+</instance>
+<instance part="VDD13" gate="G$1" x="137.16" y="25.4" smashed="yes" rot="R180">
+<attribute name="VALUE" x="136.652" y="21.59" size="1.778" layer="96" rot="R270"/>
 </instance>
 <instance part="J26" gate="J$1" x="55.88" y="132.08" smashed="yes" rot="R270">
@@
 <attribute name="VALUE" x="243.84" y="27.94" size="1.778" layer="96" rot="R90"/>
 </instance>
-<instance part="GND23" gate="1" x="137.16" y="109.22" smashed="yes">
-<attribute name="VALUE" x="138.176" y="101.6" size="1.778" layer="96" rot="R90"/>
-</instance>
-<instance part="GND24" gate="1" x="119.38" y="22.86" smashed="yes">
-<attribute name="VALUE" x="120.142" y="16.51" size="1.778" layer="96" rot="R90"/>
-</instance>
-<instance part="GND25" gate="1" x="137.16" y="22.86" smashed="yes">
-<attribute name="VALUE" x="138.176" y="16.51" size="1.778" layer="96" rot="R90"/>
+<instance part="GND23" gate="1" x="139.7" y="109.22" smashed="yes">
+<attribute name="VALUE" x="140.716" y="101.6" size="1.778" layer="96" rot="R90"/>
+</instance>
+<instance part="GND24" gate="1" x="121.92" y="22.86" smashed="yes">
+<attribute name="VALUE" x="122.682" y="16.51" size="1.778" layer="96" rot="R90"/>
+</instance>
+<instance part="GND25" gate="1" x="139.7" y="22.86" smashed="yes">
+<attribute name="VALUE" x="140.716" y="16.51" size="1.778" layer="96" rot="R90"/>
 </instance>
 <instance part="J23" gate="G$1" x="99.06" y="132.08" smashed="yes" rot="R270">
@@
 </segment>
 <segment>
-<pinref part="J12" gate="J$1" pin="2"/>
-<wire x1="137.16" y1="124.46" x2="137.16" y2="111.76" width="0.1524" layer="91"/>
-<pinref part="GND23" gate="1" pin="GND"/>
-</segment>
-<segment>
-<pinref part="J24" gate="J$1" pin="2"/>
-<wire x1="119.38" y1="38.1" x2="119.38" y2="25.4" width="0.1524" layer="91"/>
-<pinref part="GND24" gate="1" pin="GND"/>
-</segment>
-<segment>
-<pinref part="J25" gate="J$1" pin="2"/>
-<wire x1="137.16" y1="38.1" x2="137.16" y2="25.4" width="0.1524" layer="91"/>
-<pinref part="GND25" gate="1" pin="GND"/>
-</segment>
-<segment>
 <pinref part="J23" gate="G$1" pin="2"/>
 <wire x1="101.6" y1="124.46" x2="101.6" y2="111.76" width="0.1524" layer="91"/>
 <pinref part="GND26" gate="1" pin="GND"/>
+</segment>
+<segment>
+<pinref part="J12" gate="J$1" pin="3"/>
+<pinref part="GND23" gate="1" pin="GND"/>
+<wire x1="139.7" y1="124.46" x2="139.7" y2="111.76" width="0.1524" layer="91"/>
+</segment>
+<segment>
+<pinref part="J24" gate="J$1" pin="3"/>
+<pinref part="GND24" gate="1" pin="GND"/>
+<wire x1="121.92" y1="38.1" x2="121.92" y2="25.4" width="0.1524" layer="91"/>
+</segment>
+<segment>
+<pinref part="J25" gate="J$1" pin="3"/>
+<pinref part="GND25" gate="1" pin="GND"/>
+<wire x1="139.7" y1="38.1" x2="139.7" y2="25.4" width="0.1524" layer="91"/>
 </segment>
 </net>
@@
 </segment>
 <segment>
-<pinref part="J24" gate="J$1" pin="3"/>
-<wire x1="121.92" y1="38.1" x2="121.92" y2="27.94" width="0.1524" layer="91"/>
-<pinref part="VDD12" gate="G$1" pin="VDD"/>
-</segment>
-<segment>
-<pinref part="J25" gate="J$1" pin="3"/>
-<wire x1="139.7" y1="38.1" x2="139.7" y2="27.94" width="0.1524" layer="91"/>
-<pinref part="VDD13" gate="G$1" pin="VDD"/>
-</segment>
-<segment>
 <pinref part="J13" gate="J$1" pin="1"/>
 <pinref part="VDD17" gate="G$1" pin="VDD"/>
@@
 </segment>
 <segment>
-<pinref part="J12" gate="J$1" pin="3"/>
+<pinref part="J12" gate="J$1" pin="2"/>
 <pinref part="VDD7" gate="G$1" pin="VDD"/>
-<wire x1="139.7" y1="124.46" x2="139.7" y2="111.76" width="0.1524" layer="91"/>
-</segment>
-</net>
+<wire x1="137.16" y1="124.46" x2="137.16" y2="111.76" width="0.1524" layer="91"/>
+</segment>
+<segment>
+<pinref part="J24" gate="J$1" pin="2"/>
+<pinref part="VDD12" gate="G$1" pin="VDD"/>
+<wire x1="119.38" y1="38.1" x2="119.38" y2="27.94" width="0.1524" layer="91"/>
+</segment>
+<segment>
+<pinref part="J25" gate="J$1" pin="2"/>
+<pinref part="VDD13" gate="G$1" pin="VDD"/>
+<wire x1="137.16" y1="38.1" x2="137.16" y2="27.94" width="0.1524" layer="91"/>
+</segment>
+</net>

Commit message: Updates to the PCB
* Removed the power jack and replaced with a 2 wire solution
* Routing changes associated with the jack removal
* Added a new Analog channel to round out 4
* Moved some of the GPIO pins around
Parts:
- added J29: ADC-1, SparkFun-Connectors:CONN_03
- J14: value 5V_INPUT -> 5V; device SparkFun-Connectors:POWER_JACKPTH_BREAD -> SparkFun-Connectors:CONN_02
- R2, R3: value 150 -> 3.3k
- R4: value 150 -> 1k
Connections:
- removed net GPIO_11: J23.1, ONION.I2S_CLK/GPIO3
- new net C1+: J21.1, J29.1
- new net GPIO_18: J1.1, ONION.PWM0/GPIO18
- net +5V: now also J14.2; no longer J14.PWR
- net GND: now also J14.1, J21.2, J29.3; no longer J14.GND, J14.GNDBREAK
- net GPIO_13: now also J23.1; no longer J1.1
- net VDD: now also J29.2
Other:
- moved on the sheet: J14

Commit message: Updating the board to the latest
Parts:
- removed C4: 10uF, SparkFun-Capacitors:10UF-POLAR-RADIAL-2.5MM-25V-20%
- removed J28: LD1117, SparkFun-Connectors:CONN_03LONGPADS
- removed J29: ADC-1, SparkFun-Connectors:CONN_03
- removed ONION: OMEGA2+, OMEGA2_:OMEGA2+
- removed R10: 100, SparkFun-Resistors:1KOHM-HORIZ-1/4W-1%
- removed R3: 3.3k, SparkFun-Resistors:1KOHM-HORIZ-1/4W-1%
- removed R4, R5, R6, R7: 1k, SparkFun-Resistors:1KOHM-HORIZ-1/4W-1%
- removed R8, R9: 4.7k, SparkFun-Resistors:1KOHM-HORIZ-1/4W-1%
- added IC1: MCP3008, adafruit:MCP3008
- added IC2: PI Zero, Rasbperry_Pi_Zero_W:RASPBERRY_PI_ZERO_W_(V1.3)
- added LDO: LD1117V33, SparkFun-IC-Power:V_REG_LD1117VXX
- added LED1: 3.3V, adafruit:LED3MM
- added LED2: 2.0V, adafruit:LED3MM
- added Q5: 2n3904, SparkFun-DiscreteSemi:TRANS_NPN-2N3904
- added R11, R13, R14, R15, R16, R17, R18, R19: 1k, SparkFun-Resistors:1KOHM-HORIZ-1/4W-5%
- added R20: 4.7k, SparkFun-Resistors:1KOHM-HORIZ-1/4W-5%
- J11: value LD1117 -> OLED Display; device SparkFun-Connectors:CONN_03LONGPADS -> SparkFun-Connectors:CONN_03X2FEMALE
- J12: value LEVEL -> UART
- J21: value MCP3424-B -> ADC2; device SparkFun-Connectors:CONN_06SILK_FEMALE_PTH -> SparkFun-Connectors:CONN_03
- J22: value MCP3424-A -> ADC1; device SparkFun-Connectors:CONN_06SILK_FEMALE_PTH -> SparkFun-Connectors:CONN_03
- J24: value ADC-3 -> DS18B20
- J25: value ADC-4 -> ADC3
- R1: device SparkFun-Resistors:1KOHM-HORIZ-1/4W-1% -> SparkFun-Resistors:1KOHM-HORIZ-1/4W-5%
- R12: value 4.7K -> 100; device SparkFun-Resistors:1KOHM-HORIZ-1/4W-1% -> SparkFun-Resistors:1KOHM-HORIZ-1/4W-5%
- R2: value 3.3k -> 1k; device SparkFun-Resistors:1KOHM-HORIZ-1/4W-1% -> SparkFun-Resistors:1KOHM-HORIZ-1/4W-5%
Connections:
- removed net C1+: J21.1, J29.1
- removed net C2+: J12.1, J21.3
- removed net C3+: J22.3, J24.1
- removed net C4+: J22.5, J25.1
- removed net GPIO_0: ONION.I2S_SDI/GPIO0, Q1.E
- removed net GPIO_13: J23.1, ONION.UART_RX0/GPIO13
- removed net GPIO_15: ONION.GPIO15, R5.1
- removed net GPIO_16: ONION.GPIO16, R6.1
- removed net GPIO_17: ONION.GPIO17, R7.1
- removed net GPIO_18: J1.1, ONION.PWM0/GPIO18
- removed net GPIO_19: J26.1, J27.1, ONION.PWM1/GPIO19, R12.2
- removed net VCC: C4.+, J28.2, ONION.3V3_IN
- new net 1WIRE: IC2.GPIO21/SPI0_SCLK1, J24.1, J26.1, J27.1, R20.1
- new net CH0: IC1.CH0, J22.1
- new net CH1: IC1.CH1, J21.1
- new net CH2: IC1.CH2, J25.1
- new net CLK: IC1.CLK, IC2.GPIO_11/SPI0_SCLK
- new net CS: IC1./CS, IC2.GPIO_8/SPI0_CE1_N
- new net GPIO13: IC2.GPIO13/PWM1, R1.1
- new net GPIO17: IC2.GPIO_17/SPI1_CS1, R14.1
- new net GPIO18: IC2.GPIO_18/PWM0/SPI1_CS0, Q1.E
- new net GPIO22: IC2.GPIO_22, R18.1
- new net GPIO23: IC2.GPIO_23, J23.1
- new net GPIO24: IC2.GPIO_24, J1.1
- new net GPIO27: IC2.GPIO27, R16.1
- new net MISO: IC1.DOUT, IC2.GPIO_9/SPI0_MISO
- new net MOSI: IC1.DIN, IC2.GPIO_10/SPI0_MOSI
- new net N$13: Q5.B, R1.2
- new net N$14: LED2.A, R2.2
- new net N$15: LED2.C, Q5.C
- new net SIG: J13.3, R11.2
- new net UART_RX0: IC2.GPIO_15/[UART]_RXD0, J12.3
- new net UART_TX0: IC2.GPIO_14/[UART]_TXD0, J12.2
- net +5V: now also IC2.+5V1, IC2.+5V2, J11.5, LDO.IN, R13.2, R15.1, R17.1, R19.1; no longer J28.3, R10.1, R3.2, R4.2
- net GND: now also IC1.AGND, IC1.CH3, IC1.CH4, IC1.CH5, IC1.CH6, IC1.CH7, IC1.GND, IC2.GND1, IC2.GND2, IC2.GND3, IC2.GND4, IC2.GND5, IC2.GND6, IC2.GND7, IC2.GND8, J12.1, J21.3, J22.3, J24.2, LDO.GND, LED1.C, Q5.E; no longer C4.-, J12.3, J21.2, J21.4, J22.1, J22.4, J22.6, J24.3, J28.1, J29.3, ONION.GND1, ONION.GND2
- net N$1: now also LED1.A, R12.1; no longer J13.3, R1.2
- net N$11: now also R19.2; no longer R4.1
- net N$2: now also R11.1; no longer R1.1
- net N$3: now also R14.2; no longer R5.2
- net N$4: now also R13.1; no longer R10.2
- net N$5: now also R16.2; no longer R6.2
- net N$6: now also R15.2; no longer R2.2
- net N$7: now also R18.2; no longer R7.2
- net N$9: now also R17.2; no longer R3.1
- net SCL: now also IC2.GPIO_3/[I2C]_SCL, J11.2; no longer J21.6, ONION.I2C_SCL/GPIO4, R9.2
- net SDA: now also IC2.GPIO_2/[I2C]_SDA, J11.4; no longer J21.5, ONION.I2C_SDA/GPIO5, R8.2
- net VDD: now also IC1.VDD, IC1.VREF, J21.2, J24.3, LDO.OUT, R12.2, R20.2; no longer J11.2, J12.2, J24.2, J29.2, R12.1, R8.1, R9.1
